Commit message: Fix gripper folding into base and enable Physics Inspector
- Replace guessed READY_POSE with a collision-free pose: all joints at 0
  (the CAD assembly) plus a 180deg Shoulder_Rotation swivel so both arms face
  the cloth/table. Verified with the new fk_check.py FK tool (grippers settle
  ~0.15 m above the table top, in front of the bases).
- Widen Shoulder_Rotation joint limit to +/-3.3 so the 180deg pose is not on a
  hard stop; regenerate so_100_dual.urdf.
- Enable omni.physx.ui / omni.physx.supportui in setup_scene.py so the Physics
  Inspector menu action resolves (fixes "Could not find action
  show_physics_inspector").
- Add fk_check.py dev tool and document pose-picking + inspector usage in README.

Co-Authored-By: Claude Opus 4.8 <noreply@anthropic.com>

File: isaac_sim/urdf/so_100_dual.urdf (robot description, URDF)
Before this commit: robot so_100_dual, 17 links, 16 joints
Joints:
- joint left_Shoulder_Rotation: limit lower=-3.14159 upper=3.14159 effort=5 velocity=2 -> lower=-3.3 upper=3.3 effort=5 velocity=2
- joint right_Shoulder_Rotation: limit lower=-3.14159 upper=3.14159 effort=5 velocity=2 -> lower=-3.3 upper=3.3 effort=5 velocity=2

Commit message: Add STS3215 motor model and wrist UVC cameras
Physics now matches the real SO-101 actuators (Feetech STS3215):
- generate_urdf.py: joint effort/velocity set to datasheet figures
  (stall torque 2.9 N.m, no-load speed 4.7 rad/s); regenerated URDF.
- import_urdf_to_usd.py: default drive gains lowered from 1e4/1e3 to the
  realistic STS3215 control gains.
- motors.py (new, OOP): FeetechSTS3215 dataclass + SO101MotorModel that applies
  per-joint PD gains, torque ceiling and speed ceiling to the articulation at
  runtime (lighter gains for the gripper jaw).

Wrist cameras (TheRobotStudio 32x32 UVC mount):
- cameras.py (new, OOP): WristCamera spawns a UsdGeom.Camera on each arm's
  Fixed_Gripper (wrist-roll) link, aimed down the gripper approach axis, with
  FOV-derived intrinsics; optional Isaac Camera sensors for frame capture.
- setup_scene.py: spawn both cameras, apply the motor model after reset, and a
  --capture-cameras flag to create readable sensors.

config.py: new MOTOR_* / *_DRIVE_* and WRIST_CAM_* parameters.
Docs: new simulation_architecture.md explaining the whole design; README updated.

Co-Authored-By: Claude Opus 4.8 <noreply@anthropic.com>

File: isaac_sim/urdf/so_100_dual.urdf (robot description, URDF)
Before this commit: robot so_100_dual, 17 links, 16 joints
Joints:
- joint left_Elbow: limit lower=-3.14159 upper=3.14159 effort=5 velocity=2 -> lower=-3.14159 upper=3.14159 effort=2.9 velocity=4.7
- joint left_Gripper: limit lower=-0.2 upper=1.7 effort=5 velocity=2 -> lower=-0.2 upper=1.7 effort=2.9 velocity=4.7
- joint left_Shoulder_Pitch: limit lower=-3.14159 upper=3.14159 effort=5 velocity=2 -> lower=-3.14159 upper=3.14159 effort=2.9 velocity=4.7
- joint left_Shoulder_Rotation: limit lower=-3.3 upper=3.3 effort=5 velocity=2 -> lower=-3.3 upper=3.3 effort=2.9 velocity=4.7
- joint left_Wrist_Pitch: limit lower=-3.14159 upper=3.14159 effort=5 velocity=2 -> lower=-3.14159 upper=3.14159 effort=2.9 velocity=4.7
- joint left_Wrist_Roll: limit lower=-3.14159 upper=3.14159 effort=5 velocity=2 -> lower=-3.14159 upper=3.14159 effort=2.9 velocity=4.7
- joint right_Elbow: limit lower=-3.14159 upper=3.14159 effort=5 velocity=2 -> lower=-3.14159 upper=3.14159 effort=2.9 velocity=4.7
- joint right_Gripper: limit lower=-0.2 upper=1.7 effort=5 velocity=2 -> lower=-0.2 upper=1.7 effort=2.9 velocity=4.7
- joint right_Shoulder_Pitch: limit lower=-3.14159 upper=3.14159 effort=5 velocity=2 -> lower=-3.14159 upper=3.14159 effort=2.9 velocity=4.7
- joint right_Shoulder_Rotation: limit lower=-3.3 upper=3.3 effort=5 velocity=2 -> lower=-3.3 upper=3.3 effort=2.9 velocity=4.7
- joint right_Wrist_Pitch: limit lower=-3.14159 upper=3.14159 effort=5 velocity=2 -> lower=-3.14159 upper=3.14159 effort=2.9 velocity=4.7
- joint right_Wrist_Roll: limit lower=-3.14159 upper=3.14159 effort=5 velocity=2 -> lower=-3.14159 upper=3.14159 effort=2.9 velocity=4.7
