Commit message: Foldnet algorithm and deformable cloth is added

File: isaac_sim/urdf/so_100_dual_foldnet.urdf (robot description, URDF)
Before this commit: robot so_100_dual_foldnet, 19 links, 18 joints
Joints:
- joint left_tcp_joint: origin xyz=0.0101 0.0 0 rpy=0 0 0 -> xyz=0.0101 -0.106 0 rpy=0 0 0
- joint right_tcp_joint: origin xyz=0.0101 0.0 0 rpy=0 0 0 -> xyz=0.0101 -0.106 0 rpy=0 0 0
